Commit message: now the test works but the next step is gonna make it move to the correct directions, idk what i exatly did, i been leaving and coming back so I think is good i guess ????? LOL

File: test.urdf (robot description, URDF)
Before this commit: robot canadarm3_large, 22 links, 21 joints
Links:
- removed link link_10
- removed link link_11
- removed link link_12
- removed link link_13
- removed link link_14
- removed link link_15
- removed link link_16
- removed link link_17
- removed link link_18
- removed link link_19
- removed link link_20
- removed link link_21
- removed link link_9
- link link_1: mass 0.8 -> 0.7
- link link_2: mass 0.8 -> 0.4
- link link_3: mass 0.7 -> 0.35; geometry collision mesh filename=test/canadarm3_large(1)(1)(1)/canadarm3_large(1)(1) - canad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; visual mesh filename=test/canadarm3_large(1)(1)(1)/canadarm3_large(1)(1) - canad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
- link link_4: mass 0.7 -> 0.5
- link link_5: mass 0.6 -> 0.35; geometry collision mesh filename=test/canadarm3_large(1)(1)(1)/canadarm3_large(1)(1) - canad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; visual mesh filename=test/canadarm3_large(1)(1)(1)/canadarm3_large(1)(1) - canad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
- link link_6: mass 0.6 -> 0.35; geometry collision mesh filename=test/canadarm3_large(1)(1)(1)/canadarm3_large(1)(1) - canad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; visual mesh filename=test/canadarm3_large(1)(1)(1)/canadarm3_large(1)(1) - canad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
- link link_7: mass 0.5 -> 0.35; geometry collision mesh filename=test/canadarm3_large(1)(1)(1)/canadarm3_large(1)(1) - canad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; visual mesh filename=test/canadarm3_large(1)(1)(1)/canadarm3_large(1)(1) - canad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
- link link_8: mass 0.5 -> 0.3
Joints:
- removed joint joint_1
- removed joint joint_10
- removed joint joint_11
- removed joint joint_12
- removed joint joint_13
- removed joint joint_14
- removed joint joint_15
- removed joint joint_2
- removed joint joint_21
- removed joint joint_4
- removed joint joint_6
- removed joint joint_8
- removed joint joint_9
- joint joint_16: child link_16 -> link_4; limit lower=-3.1416 upper=3.1416 effort=100 velocity=1 -> lower=-3.124 upper=3.124 effort=100 velocity=1; origin xyz=0 0 0 rpy=0 0 0 -> xyz=0.01 0.01 0.01 rpy=0 0 0; parent link_15 -> link_3
- joint joint_17: child link_17 -> link_5; limit lower=-3.1416 upper=3.1416 effort=100 velocity=1 -> lower=-3.124 upper=3.124 effort=100 velocity=1; origin xyz=0 0 0 rpy=0 0 0 -> xyz=0.01 0.01 0.01 rpy=0 0 0; parent link_16 -> link_4
- joint joint_18: child link_18 -> link_6; limit lower=-3.1416 upper=3.1416 effort=100 velocity=1 -> lower=-3.124 upper=3.124 effort=100 velocity=1; origin xyz=0 0 0 rpy=0 0 0 -> xyz=0.01 0.01 0.01 rpy=0 0 0; parent link_17 -> link_5
- joint joint_19: child link_19 -> link_7; limit lower=-3.1416 upper=3.1416 effort=100 velocity=1 -> lower=-3.124 upper=3.124 effort=100 velocity=1; origin xyz=0 0 0 rpy=0 0 0 -> xyz=0.01 0.01 0.01 rpy=0 0 0; parent link_18 -> link_6
- joint joint_20: child link_20 -> link_8; limit lower=-3.1416 upper=3.1416 effort=100 velocity=1 -> lower=-3.124 upper=3.124 effort=100 velocity=1; origin xyz=0 0 0 rpy=0 0 0 -> xyz=0.01 0.01 0.01 rpy=0 0 0; parent link_19 -> link_7
- joint joint_3: child link_3 -> link_1; limit lower=-3.1416 upper=3.1416 effort=100 velocity=1 -> lower=-3.124 upper=3.124 effort=100 velocity=1; origin xyz=0 0 0 rpy=0 0 0 -> xyz=0.01 0.01 0.01 rpy=0 0 0; parent link_2 -> base_link
- joint joint_5: child link_5 -> link_2; limit lower=-3.1416 upper=3.1416 effort=100 velocity=1 -> lower=-3.124 upper=3.124 effort=100 velocity=1; origin xyz=0 0 0 rpy=0 0 0 -> xyz=0.01 0.01 0.01 rpy=0 0 0; parent link_4 -> link_1
- joint joint_7: child link_7 -> link_3; limit lower=-3.1416 upper=3.1416 effort=100 velocity=1 -> lower=-3.124 upper=3.124 effort=100 velocity=1; origin xyz=0 0 0 rpy=0 0 0 -> xyz=0.01 0.01 0.01 rpy=0 0 0; parent link_6 -> link_2

Commit message: clean the names of things

File: test.urdf (robot description, URDF)
Before this commit: robot canadarm3_large, 9 links, 8 joints
Links:
- link base_link: geometry collision mesh filename=test/canadarm3_large/canadarm3_0 - Surface 1.stl; visual mesh filename=test/canadarm3_large/canadarm3_0 - Surface 1.stl
- link link_1: geometry collision mesh filename=test/canadarm3_large/canadarm3_1 - Surface 1.stl; visual mesh filename=test/canadarm3_large/canadarm3_1 - Surface 1.stl
- link link_2: geometry collision mesh filename=test/canadarm3_large/canadarm3_2 - Surface 1.stl; visual mesh filename=test/canadarm3_large/canadarm3_2 - Surface 1.stl
- link link_3: geometry collision mesh filename=test/canadarm3_large/canadarm3_3 - Surface 1.stl; visual mesh filename=test/canadarm3_large/canadarm3_3 - Surface 1.stl
- link link_4: geometry collision mesh filename=test/canadarm3_large/canadarm3_4 - Surface 1.stl; visual mesh filename=test/canadarm3_large/canadarm3_4 - Surface 1.stl
- link link_5: geometry collision mesh filename=test/canadarm3_large/canadarm3_5 - Surface 1.stl; visual mesh filename=test/canadarm3_large/canadarm3_5 - Surface 1.stl
- link link_6: geometry collision mesh filename=test/canadarm3_large/canadarm3_6 - Surface 1.stl; visual mesh filename=test/canadarm3_large/canadarm3_6 - Surface 1.stl
- link link_7: geometry collision mesh filename=test/canadarm3_large/canadarm3_7 - Surface 1.stl; visual mesh filename=test/canadarm3_large/canadarm3_7 - Surface 1.stl
- link link_8: geometry collision mesh filename=test/canadarm3_large/canadarm3_8 - Surface 1.stl; visual mesh filename=test/canadarm3_large/canadarm3_8 - Surface 1.stl
Joints:
- removed joint joint_16
- removed joint joint_17
- removed joint joint_18
- removed joint joint_19
- removed joint joint_20
- added joint joint_1: type revolute, parent base_link, child link_1, origin xyz=0.01 0.01 0.01 rpy=0 0 0, axis 0 1 0, limit lower=-3.124 upper=3.124 effort=100 velocity=1
- added joint joint_2: type revolute, parent link_1, child link_2, origin xyz=0.01 0.01 0.01 rpy=0 0 0, axis 0 1 0, limit lower=-3.124 upper=3.124 effort=100 velocity=1
- added joint joint_4: type revolute, parent link_3, child link_4, origin xyz=0.01 0.01 0.01 rpy=0 0 0, axis 1 0 0, limit lower=-3.124 upper=3.124 effort=100 velocity=1
- added joint joint_6: type revolute, parent link_5, child link_6, origin xyz=0.01 0.01 0.01 rpy=0 0 0, axis 1 0 0, limit lower=-3.124 upper=3.124 effort=100 velocity=1
- added joint joint_8: type revolute, parent link_7, child link_8, origin xyz=0.01 0.01 0.01 rpy=0 0 0, axis 0 0 1, limit lower=-3.124 upper=3.124 effort=100 velocity=1
- joint joint_3: axis 0 1 0 -> 0 0 1; child link_1 -> link_3; parent base_link -> link_2
- joint joint_5: child link_2 -> link_5; parent link_1 -> link_4
- joint joint_7: axis 0 0 1 -> 0 1 0; child link_3 -> link_7; parent link_2 -> link_6
