Commit message: fix color, fix radius of the arm, fix limits(estimation) add collition and order every link by visual, collision, inertial. Next step is add the estimated length and mass + fix the origins

File: arm.urdf (robot description, URDF)
Before this commit: robot 7jointed_arm, 9 links, 8 joints
Links:
- link base_link: geometry collision box size=1 1 .01; visual box size=1 1 .01
- link elbow_link: geometry collision cylinder length=0.25 radius=0.23; visual cylinder length=0.25 radius=0.23
- link end_effector: geometry collision sphere radius=0.05; visual sphere radius=0.05
- link shoulder_link_1: geometry collision cylinder length=0.2 radius=0.23; visual cylinder length=0.2 radius=0.23
- link shoulder_link_2: geometry collision cylinder length=0.2 radius=0.23; visual cylinder length=0.2 radius=0.23
- link shoulder_link_3: geometry collision cylinder length=0.2 radius=0.23; visual cylinder length=0.2 radius=0.23
- link wrist_link_1: geometry collision cylinder length=0.15 radius=0.23; visual cylinder length=0.15 radius=0.23
- link wrist_link_2: geometry collision cylinder length=0.15 radius=0.23; visual cylinder length=0.15 radius=0.23
- link wrist_link_3: geometry collision cylinder length=0.15 radius=0.23; visual cylinder length=0.15 radius=0.23
Joints:
- joint shoulder_joint_1: limit lower=-1.57 upper=1.57 effort=100 velocity=1 -> lower=-3.124 upper=3.124 effort=100 velocity=1
- joint shoulder_joint_3: limit lower=-1.57 upper=1.57 effort=100 velocity=1 -> lower=-3.14 upper=3.14 effort=100 velocity=1
- joint wrist_joint_1: limit lower=-1.57 upper=1.57 effort=50 velocity=1 -> lower=-3.14 upper=3.14 effort=50 velocity=1
- joint wrist_joint_3: limit lower=-1.57 upper=1.57 effort=50 velocity=1 -> lower=-3.14 upper=3.14 effort=50 velocity=1

Commit message: add guessed dimentions, next:

File: arm.urdf (robot description, URDF)
Before this commit: robot 7jointed_arm, 9 links, 8 joints
Links:
- link base_link: geometry collision box size=1 1 .1; visual box size=1 1 .1
- link elbow_link: geometry collision cylinder length=0.01 radius=0.01; visual cylinder length=0.01 radius=0.01
- link end_effector: geometry collision sphere radius=0.25; visual sphere radius=0.25
- link shoulder_link_1: geometry collision box size=0.37427 0.37427 .44090; visual box size=0.37427 0.37427 .44090
- link shoulder_link_2: geometry collision box size=0.38129 0.36253 0.35895; visual box size=0.38129 0.36253 0.35895
- link shoulder_link_3: geometry collision box size=0.33712 0.27699 0.38135; visual box size=0.33712 0.27699 0.38135
- link wrist_link_1: geometry collision box size=0.33712 0.27699 0.38135; visual box size=0.33712 0.27699 0.38135
- link wrist_link_2: geometry collision box size=0.38129 0.36253 0.35895; visual box size=0.38129 0.36253 0.35895
- link wrist_link_3: geometry collision box size=0.37427 0.37427 .44090; visual box size=0.37427 0.37427 .44090

Commit message: set origin of shoulder link 1 on the base, also change base to be a 2D plane :)

File: arm.urdf (robot description, URDF)
Before this commit: robot 7jointed_arm, 9 links, 8 joints
Links:
- link base_link: geometry collision box size=1 1 0; visual box size=1 1 0
Joints:
- joint shoulder_joint_1: origin xyz=0 0 0.1 rpy=0 0 0 -> xyz=0 0 0.22090 rpy=0 0 0

Commit message: set origin of shoulder link 2 at the end of shoulder link 1

File: arm.urdf (robot description, URDF)
Before this commit: robot 7jointed_arm, 9 links, 8 joints
Joints:
- joint shoulder_joint_2: origin xyz=0 0 0.2 rpy=0 0 0 -> xyz=0 0 0.4 rpy=0 0 0

Commit message: fix the .stl files so their center point is the rotation axis, and their origin and rotation axis in arm.urdf file, Also add a commented version for future testing where each part is fixed in 1 position

File: arm.urdf (robot description, URDF)
Before this commit: robot 7jointed_arm, 9 links, 8 joints
Links:
- removed link elbow_link
- removed link end_effector
- removed link shoulder_link_1
- removed link shoulder_link_2
- removed link shoulder_link_3
- removed link wrist_link_1
- removed link wrist_link_2
- removed link wrist_link_3
- added link link_1, mass 0.7; collision mesh filename=test/canadarm3_large/canadarm3_1 - Surface 1.stl; visual mesh filename=test/canadarm3_large/canadarm3_1 - Surface 1.stl
- added link link_2, mass 0.4; collision mesh filename=test/canadarm3_large/canadarm3_2 - Surface 1.stl; visual mesh filename=test/canadarm3_large/canadarm3_2 - Surface 1.stl
- added link link_3, mass 0.35; collision mesh filename=test/canadarm3_large/canadarm3_3 - Surface 1.stl; visual mesh filename=test/canadarm3_large/canadarm3_3 - Surface 1.stl
- added link link_4, mass 0.5; collision mesh filename=test/canadarm3_large/canadarm3_4 - Surface 1.stl; visual mesh filename=test/canadarm3_large/canadarm3_4 - Surface 1.stl
- added link link_5, mass 0.35; collision mesh filename=test/canadarm3_large/canadarm3_5 - Surface 1.stl; visual mesh filename=test/canadarm3_large/canadarm3_5 - Surface 1.stl
- added link link_6, mass 0.35; collision mesh filename=test/canadarm3_large/canadarm3_6 - Surface 1.stl; visual mesh filename=test/canadarm3_large/canadarm3_6 - Surface 1.stl
- added link link_7, mass 0.35; collision mesh filename=test/canadarm3_large/canadarm3_7 - Surface 1.stl; visual mesh filename=test/canadarm3_large/canadarm3_7 - Surface 1.stl
- added link link_8, mass 0.3; collision mesh filename=test/canadarm3_large/canadarm3_8 - Surface 1.stl; visual mesh filename=test/canadarm3_large/canadarm3_8 - Surface 1.stl
- link base_link: mass 1 -> 1.0; geometry collision mesh filename=test/canadarm3_large/canadarm3_0 - Surface 1.stl; visual mesh filename=test/canadarm3_large/canadarm3_0 - Surface 1.stl
Joints:
- removed joint elbow_joint
- removed joint end_effector_joint
- removed joint shoulder_joint_1
- removed joint shoulder_joint_2
- removed joint shoulder_joint_3
- removed joint wrist_joint_1
- removed joint wrist_joint_2
- removed joint wrist_joint_3
- added joint joint_1: type revolute, parent base_link, child link_1, origin xyz=0.01 0.01 0.01 rpy=0 0 0, axis 0 0 1, limit lower=-6.248 upper=6.248 effort=100 velocity=1
- added joint joint_2: type revolute, parent link_1, child link_2, origin xyz=-(0.19518290-(0.39036581/2)) -(19590171-(0.37290171/2)) 0.613788085 rpy=0 0 0, axis 0 1 0, limit lower=-6.248 upper=6.248 effort=100 velocity=1
- added joint joint_3: type revolute, parent link_2, child link_3, origin xyz=0.025 -0.345 (-0.592-0.613788085) rpy=0 0 0, axis 0 1 0, limit lower=-6.248 upper=6.248 effort=100 velocity=1
- added joint joint_4: type revolute, parent link_3, child link_4, origin xyz=0.323 (-0.33-0.345) (0.592-1.205788085) rpy=0 0 0, axis 1 0 0, limit lower=-6.248 upper=6.248 effort=100 velocity=1
- added joint joint_5: type revolute, parent link_4, child link_5, origin xyz=0.37 (-0.33-0.345) 3.646211915 rpy=0 0 0, axis 1 0 0, limit lower=-6.248 upper=6.248 effort=100 velocity=1
- added joint joint_6: type revolute, parent link_5, child link_6, origin xyz=.335 (-0.33-0.345) -3.646211915 rpy=0 0 0, axis 1 0 0, limit lower=-6.248 upper=6.248 effort=100 velocity=1
- added joint joint_7: type revolute, parent link_6, child link_7, origin xyz=0.0 -0.345 0.0 rpy=0 0 0, axis 0 1 0, limit lower=-6.248 upper=6.248 effort=100 velocity=1
- added joint joint_8: type revolute, parent link_7, child link_8, origin xyz=0.01 0.01 -0.613788085 rpy=0 0 0, axis 0 0 1, limit lower=-6.248 upper=6.248 effort=100 velocity=1

Commit message: move the go_to.py file to a separeted folder called Movement and move the Canadarm3 stl files to a separeted folder outside test folder and deleate test folder to avoid confusions

File: arm.urdf (robot description, URDF)
Before this commit: robot canadarm3_large, 9 links, 8 joints
Links:
- link base_link: geometry collision mesh filename=canadarm3_large/canadarm3_0 - Surface 1.stl; visual mesh filename=canadarm3_large/canadarm3_0 - Surface 1.stl
- link link_1: geometry collision mesh filename=canadarm3_large/canadarm3_1 - Surface 1.stl; visual mesh filename=canadarm3_large/canadarm3_1 - Surface 1.stl
- link link_2: geometry collision mesh filename=canadarm3_large/canadarm3_2 - Surface 1.stl; visual mesh filename=canadarm3_large/canadarm3_2 - Surface 1.stl
- link link_3: geometry collision mesh filename=canadarm3_large/canadarm3_3 - Surface 1.stl; visual mesh filename=canadarm3_large/canadarm3_3 - Surface 1.stl
- link link_4: geometry collision mesh filename=canadarm3_large/canadarm3_4 - Surface 1.stl; visual mesh filename=canadarm3_large/canadarm3_4 - Surface 1.stl
- link link_5: geometry collision mesh filename=canadarm3_large/canadarm3_5 - Surface 1.stl; visual mesh filename=canadarm3_large/canadarm3_5 - Surface 1.stl
- link link_6: geometry collision mesh filename=canadarm3_large/canadarm3_6 - Surface 1.stl; visual mesh filename=canadarm3_large/canadarm3_6 - Surface 1.stl
- link link_7: geometry collision mesh filename=canadarm3_large/canadarm3_7 - Surface 1.stl; visual mesh filename=canadarm3_large/canadarm3_7 - Surface 1.stl
- link link_8: geometry collision mesh filename=canadarm3_large/canadarm3_8 - Surface 1.stl; visual mesh filename=canadarm3_large/canadarm3_8 - Surface 1.stl

Commit message: Fix a bug that i didn't notice until now, joint 3 was moving in the wrong axis, fixed this by making the first joint aFixed joint instead of a revolute and chaniging the axis on the 3rd joint, now theres a new problem that the camera output is sending incorrect mesurements, i belive is because i set the position to the last joint but now that is fixed is wrong, also I should deleate the base link because is waisting resources and is litteraly doing nothing. so goal for next commit is deleting the base_link and the first joint. After that is fixing camera output

File: arm.urdf (robot description, URDF)
Before this commit: robot canadarm3_large, 9 links, 8 joints
Joints:
- joint joint_1: axis 0 0 1 -> (none); limit lower=-6.248 upper=6.248 effort=100 velocity=1 -> (none); type revolute -> fixed
- joint joint_2: axis 0 1 0 -> 0 0 1; limit lower=-6.248 upper=6.248 effort=100 velocity=1 -> lower=-3.124 upper=3.124 effort=100 velocity=1
- joint joint_3: limit lower=-6.248 upper=6.248 effort=100 velocity=1 -> lower=-3.124 upper=3.124 effort=100 velocity=1
- joint joint_4: limit lower=-6.248 upper=6.248 effort=100 velocity=1 -> lower=-3.124 upper=3.124 effort=100 velocity=1
- joint joint_5: limit lower=-6.248 upper=6.248 effort=100 velocity=1 -> lower=-3.124 upper=3.124 effort=100 velocity=1
- joint joint_6: limit lower=-6.248 upper=6.248 effort=100 velocity=1 -> lower=-3.124 upper=3.124 effort=100 velocity=1
- joint joint_7: limit lower=-6.248 upper=6.248 effort=100 velocity=1 -> lower=-3.124 upper=3.124 effort=100 velocity=1
- joint joint_8: limit lower=-6.248 upper=6.248 effort=100 velocity=1 -> lower=-3.124 upper=3.124 effort=100 velocity=1

Commit message: Delete the Base link that did't do anything

File: arm.urdf (robot description, URDF)
Before this commit: robot canadarm3_large, 9 links, 8 joints
Links:
- removed link base_link
Joints:
- removed joint joint_1

Commit message: fix the arm.urdf file so it looks better

File: arm.urdf (robot description, URDF)
Before this commit: robot canadarm3_large, 8 links, 7 joints
Joints:
- removed joint joint_8
- added joint joint_1: type revolute, parent link_1, child link_2, origin xyz=0 0 0.613788085 rpy=0 0 0, axis 0 0 1, limit lower=-3.124 upper=3.124 effort=100 velocity=1
- joint joint_2: axis 0 0 1 -> 0 1 0; child link_2 -> link_3; origin xyz=-(0.19518290-(0.39036581/2)) -(19590171-(0.37290171/2)) 0.613788085 rpy=0 0 0 -> xyz=0.0 -0.345 0.0 rpy=0 0 0; parent link_1 -> link_2
- joint joint_3: axis 0 1 0 -> 1 0 0; child link_3 -> link_4; origin xyz=0.025 -0.345 (-0.592-0.613788085) rpy=0 0 0 -> xyz=0.323 0.0 0.0 rpy=0 0 0; parent link_2 -> link_3
- joint joint_4: child link_4 -> link_5; origin xyz=0.323 (-0.33-0.345) (0.592-1.205788085) rpy=0 0 0 -> xyz=0.37 0.0 3.646211915 rpy=0 0 0; parent link_3 -> link_4
- joint joint_5: child link_5 -> link_6; origin xyz=0.37 (-0.33-0.345) 3.646211915 rpy=0 0 0 -> xyz=0.335 0.0 -3.646211915 rpy=0 0 0; parent link_4 -> link_5
- joint joint_6: axis 1 0 0 -> 0 1 0; child link_6 -> link_7; origin xyz=.335 (-0.33-0.345) -3.646211915 rpy=0 0 0 -> xyz=0.0 -0.345 0.0 rpy=0 0 0; parent link_5 -> link_6
- joint joint_7: axis 0 1 0 -> 0 0 1; child link_7 -> link_8; origin xyz=0.0 -0.345 0.0 rpy=0 0 0 -> xyz=0.0 0.0 -0.613788085 rpy=0 0 0; parent link_6 -> link_7
